File: tinycraft.kicad_sch (KiCad schematic)
At the start: 38 parts, among them J1 USB_C_Receptacle_USB2.0_16P, J2 UART, J3 u.FL, SW1 BOOT, U1 ESP32-S3, U2 CH221K, U3 AMS1117-3.3, U4 W25Q16JVSS, Y1 40MHz +- 10ppm

Commit message: upload 2
Parts:
- added C19: 100nF, Capacitor_SMD:C_0402_1005Metric, symbol Device:C_Small
- C3: value 10uF -> 22uF; footprint Capacitor_SMD:C_0402_1005Metric -> Capacitor_Tantalum_SMD:CP_EIA-3216-18_Kemet-A
- C4, C5: value TBD -> 12pF
- L1: value TBD -> 24nH
- R1: value 510R -> 1K; footprint Resistor_SMD:R_0402_1005Metric -> Resistor_SMD:R_1206_3216Metric
- Y1: value 40MHz +- 10ppm -> HCI 0132M4-40.000F10FTNN
Connections:
- net +3V3: now also C19.2
- net GND: now also C19.1
Changed lines of the file:
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@@
 	)
 	(junction
+		(at 55.88 157.48)
+		(diameter 0)
+		(color 0 0 0 0)
+	)
+	(junction
 		(at 236.22 250.19)
 		(diameter 0)
@@
 	)
 	(junction
-		(at 55.88 149.86)
+		(at 66.04 149.86)
 		(diameter 0)
 		(color 0 0 0 0)
@@
 	)
 	(junction
+		(at 55.88 149.86)
+		(diameter 0)
+		(color 0 0 0 0)
+	)
+	(junction
 		(at 190.5 175.26)
 		(diameter 0)
@@
 	(wire
 		(pts
+			(xy 66.04 154.94) (xy 66.04 157.48)
+		)
+		(stroke
+			(width 0)
+			(type default)
+		)
+	)
+	(wire
+		(pts
 			(xy 54.61 38.1) (xy 73.66 38.1)
 		)
@@
 	(wire
 		(pts
+			(xy 55.88 157.48) (xy 66.04 157.48)
+		)
+		(stroke
+			(width 0)
+			(type default)
+		)
+	)
+	(wire
+		(pts
 			(xy 246.38 196.85) (xy 246.38 189.23)
 		)
@@
 	(wire
 		(pts
+			(xy 55.88 149.86) (xy 66.04 149.86)
+		)
+		(stroke
+			(width 0)
+			(type default)
+		)
+	)
+	(wire
+		(pts
 			(xy 190.5 158.75) (xy 190.5 165.1)
 		)
@@
 	(symbol
 		(lib_id "power:+3V3")
-		(at 55.88 149.86 0)
+		(at 66.04 149.86 0)
 		(unit 1)
 		(body_style 1)
@@
 		(dnp no)
 		(property "Reference" "#PWR06"
-			(at 55.88 153.67 0)
+			(at 66.04 153.67 0)
 			(hide yes)
 			(show_name no)
@@
 		)
 		(property "Value" "+3V3"
-			(at 59.436 148.59 0)
+			(at 69.596 148.59 0)
 			(show_name no)
 			(do_not_autoplace no)
@@
 		)
 		(property "Footprint" ""
-			(at 55.88 149.86 0)
+			(at 66.04 149.86 0)
 			(hide yes)
 			(show_name no)
@@
 		)
 		(property "Datasheet" ""
-			(at 55.88 149.86 0)
+			(at 66.04 149.86 0)
 			(hide yes)
 			(show_name no)
@@
 		)
 		(property "Description" "Power symbol creates a global label with name \"+3V3\""
-			(at 55.88 149.86 0)
+			(at 66.04 149.86 0)
 			(hide yes)
 			(show_name no)
@@
 			)
 		)
-		(property "Value" "TBD"
+		(property "Value" "12pF"
 			(at 116.332 246.126 90)
 			(show_name no)
@@
 			)
 		)
-		(property "Value" "10uF"
+		(property "Value" "22uF"
 			(at 58.42 153.67 0)
 			(show_name no)
@@
 			)
 		)
-		(property "Footprint" "Capacitor_SMD:C_0402_1005Metric"
+		(property "Footprint" "Capacitor_Tantalum_SMD:CP_EIA-3216-18_Kemet-A"
 			(at 55.88 152.4 0)
 			(hide yes)
@@
 		(dnp no)
 		(property "Reference" "Y1"
-			(at 144.272 241.3 90)
+			(at 147.828 240.03 90)
 			(show_name no)
 			(do_not_autoplace no)
@@
 			)
 		)
-		(property "Value" "40MHz +- 10ppm"
-			(at 144.272 243.3321 90)
+		(property "Value" "HCI 0132M4-40.000F10FTNN"
+			(at 147.828 242.0621 90)
 			(show_name no)
 			(do_not_autoplace no)
@@
 	(symbol
 		(lib_id "Device:C_Small")
+		(at 66.04 152.4 180)
+		(unit 1)
+		(body_style 1)
+		(exclude_from_sim no)
+		(in_bom yes)
+		(on_board yes)
+		(in_pos_files yes)
+		(dnp no)
+		(property "Reference" "C19"
+			(at 68.58 151.13 0)
+			(show_name no)
+			(do_not_autoplace no)
+			(effects
+				(font
+					(size 1.27 1.27)
+				)
+				(justify right)
+			)
+		)
+		(property "Value" "100nF"
+			(at 68.58 153.67 0)
+			(show_name no)
+			(do_not_autoplace no)
+			(effects
+				(font
+					(size 1.27 1.27)
+				)
+				(justify right)
+			)
+		)
+		(property "Footprint" "Capacitor_SMD:C_0402_1005Metric"
+			(at 66.04 152.4 0)
+			(hide yes)
+			(show_name no)
+			(do_not_autoplace no)
+			(effects
+				(font
+					(size 1.27 1.27)
+				)
+			)
+		)
+		(property "Datasheet" ""
+			(at 66.04 152.4 0)
+			(hide yes)
+			(show_name no)
+			(do_not_autoplace no)
+			(effects
+				(font
+					(size 1.27 1.27)
+				)
+			)
+		)
+		(property "Description" "Unpolarized capacitor, small symbol"
+			(at 66.04 152.4 0)
+			(hide yes)
+			(show_name no)
+			(do_not_autoplace no)
+			(effects
+				(font
+					(size 1.27 1.27)
+				)
+			)
+		)
+		(pin "1"
+		)
+		(pin "2"
+		)
+		(instances
+			(project "tinycraft"
+				(path "/d68ae6e2-3c29-4df4-84fb-847711267fbc"
+					(reference "C19")
+					(unit 1)
+				)
+			)
+		)
+	)
+	(symbol
+		(lib_id "Device:C_Small")
 		(at 238.76 226.06 0)
 		(unit 1)
@@
 			)
 		)
-		(property "Value" "TBD"
+		(property "Value" "24nH"
 			(at 151.13 245.11 90)
 			(show_name no)
@@
 			)
 		)
-		(property "Value" "TBD"
+		(property "Value" "12pF"
 			(at 116.586 254 90)
 			(show_name no)
@@
 			)
 		)
-		(property "Value" "510R"
+		(property "Value" "1K"
 			(at 69.85 30.48 90)
 			(show_name no)
@@
 			)
 		)
-		(property "Footprint" "Resistor_SMD:R_0402_1005Metric"
+		(property "Footprint" "Resistor_SMD:R_1206_3216Metric"
 			(at 69.85 33.02 0)
 			(hide yes)
